File: cartprotoboard.sch (KiCad schematic (older format))
At the start: 7 parts, among them CON1 Conn_02x20_Odd_Even, U1 W25Q128JVSIQ

Commit message: Add notes
Other:
- note added: "Notes:\n- U1 can be any serial flash chip compatible with the Lattice ECP5 FPGA \n series. Something with 4MiB >= size >= 16MiB is preferred.\n- Max power draw from 3V3: 500mA\n- Max power draw from 5V: 300mA\n- Max draw from Vbat: whatever the batteries can supply\n- Note that 5V is generated by a boost converter from the battery \n voltage, it is NOT the 5V USB line.\n- CON1 connects to the bad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"
Changed lines of the file:
@@
 Wire Wire Line
 	5200 3350 5200 3250
+Text Notes 5500 2200 0    50   ~ 0
+Notes:\n- U1 can be any serial flash chip compatible with the Lattice ECP5 FPGA \n  series. Something with 4MiB >= size >= 16MiB is preferred.\n- Max power draw from 3V3: 500mA\n- Max power draw from 5V: 300mA\n- Max draw from Vbat: whatever the batteries can supply\n- Note that 5V is generated by a boost converter from the battery \n  voltage, it is NOT the 5V USB line.\n- CON1 connects to the badge, HDR1 is an empty header you can solder\n  wires to
 $EndSCHEMATC
