File: cartprotoboard.kicad_pcb (KiCad board)
At the start: 2 copper layers, 80.2 x 62.8 mm, 488 parts, among them CON1 PinHeader_2x20_P2.54mm_Horizo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, U1 SSOP-8_5.25x5.24mm_P1.27mm

Commit message: Final board
Parts:
- C1, C2, C3, C4: value C_0603_1608Metric -> 100n
- CON1: value PinHeader_2x20_P2.54mm_Horizontal_Mirrored -> Conn_02x20_Odd_Even
- HDR1: value PinHeader_2x20_P2.54mm_Vertical_virt -> Conn_02x20_Odd_Even
- U1: value SSOP-8_5.25x5.24mm_P1.27mm -> W25Q128JVSIQ
- turned C1 to 0 degrees
- turned C2 to 270 degrees
- turned C3 to 270 degrees
- turned C4 to 270 degrees
Connections:
- C1 pad 1: (no net) -> 3V3
- C1 pad 2: (no net) -> GND
- C2 pad 1: (no net) -> 3V3
- C2 pad 2: (no net) -> GND
- C3 pad 1: (no net) -> VBAT
- C3 pad 2: (no net) -> GND
- C4 pad 1: (no net) -> 5V
- C4 pad 2: (no net) -> GND
- CON1 pad 1: (no net) -> 3V3
- CON1 pad 10: (no net) -> GENIO2
- CON1 pad 11: (no net) -> GENIO3
- CON1 pad 12: (no net) -> GENIO4
- CON1 pad 13: (no net) -> GENIO5
- CON1 pad 14: (no net) -> GENIO6
- CON1 pad 15: (no net) -> GENIO7
- CON1 pad 16: (no net) -> GENIO8
- CON1 pad 17: (no net) -> GENIO9
- CON1 pad 18: (no net) -> GENIO10
- CON1 pad 19: (no net) -> GENIO11
- CON1 pad 2: (no net) -> GND
- CON1 pad 20: (no net) -> GENIO12
- CON1 pad 21: (no net) -> GENIO13
- CON1 pad 22: (no net) -> GENIO14
- CON1 pad 23: (no net) -> GENIO15
- CON1 pad 24: (no net) -> GENIO16
- CON1 pad 25: (no net) -> GENIO17
- CON1 pad 26: (no net) -> GENIO18
- CON1 pad 27: (no net) -> GENIO19
- CON1 pad 28: (no net) -> GENIO20
- CON1 pad 29: (no net) -> GENIO21
- CON1 pad 3: (no net) -> CS
- CON1 pad 30: (no net) -> GENIO22
- CON1 pad 31: (no net) -> GENIO23
- CON1 pad 32: (no net) -> GENIO24
- CON1 pad 33: (no net) -> GENIO25
- CON1 pad 34: (no net) -> GENIO26
- CON1 pad 35: (no net) -> GENIO27
- CON1 pad 36: (no net) -> GENIO28
- CON1 pad 37: (no net) -> GENIO29
- CON1 pad 38: (no net) -> GENIO30
- CON1 pad 39: (no net) -> VBAT
- CON1 pad 4: (no net) -> HOLD
- CON1 pad 40: (no net) -> 5V
- CON1 pad 5: (no net) -> MISO
- CON1 pad 6: (no net) -> SCK
- CON1 pad 7: (no net) -> WP
- CON1 pad 8: (no net) -> MOSI
- CON1 pad 9: (no net) -> GENIO1
- HDR1 pad 1: (no net) -> 3V3
- HDR1 pad 10: (no net) -> GENIO2
- HDR1 pad 11: (no net) -> GENIO3
- HDR1 pad 12: (no net) -> GENIO4
- HDR1 pad 13: (no net) -> GENIO5
- HDR1 pad 14: (no net) -> GENIO6
- HDR1 pad 15: (no net) -> GENIO7
- HDR1 pad 16: (no net) -> GENIO8
- HDR1 pad 17: (no net) -> GENIO9
- HDR1 pad 18: (no net) -> GENIO10
- HDR1 pad 19: (no net) -> GENIO11
- HDR1 pad 2: (no net) -> GND
- HDR1 pad 20: (no net) -> GENIO12
- HDR1 pad 21: (no net) -> GENIO13
- HDR1 pad 22: (no net) -> GENIO14
- HDR1 pad 23: (no net) -> GENIO15
- HDR1 pad 24: (no net) -> GENIO16
- HDR1 pad 25: (no net) -> GENIO17
- HDR1 pad 26: (no net) -> GENIO18
- HDR1 pad 27: (no net) -> GENIO19
- HDR1 pad 28: (no net) -> GENIO20
- HDR1 pad 29: (no net) -> GENIO21
- HDR1 pad 3: (no net) -> 3V3
- HDR1 pad 30: (no net) -> GENIO22
- HDR1 pad 31: (no net) -> GENIO23
- HDR1 pad 32: (no net) -> GENIO24
- HDR1 pad 33: (no net) -> GENIO25
- HDR1 pad 34: (no net) -> GENIO26
- HDR1 pad 35: (no net) -> GENIO27
- HDR1 pad 36: (no net) -> GENIO28
- HDR1 pad 37: (no net) -> GENIO29
- HDR1 pad 38: (no net) -> GENIO30
- HDR1 pad 39: (no net) -> VBAT
- HDR1 pad 4: (no net) -> GND
- HDR1 pad 40: (no net) -> 5V
- HDR1 pad 5: (no net) -> 3V3
- HDR1 pad 6: (no net) -> GND
- HDR1 pad 7: (no net) -> 3V3
- HDR1 pad 8: (no net) -> GND
- HDR1 pad 9: (no net) -> GENIO1
- U1 pad 1: (no net) -> CS
- U1 pad 2: (no net) -> MISO
- U1 pad 3: (no net) -> WP
- U1 pad 4: (no net) -> GND
- U1 pad 5: (no net) -> MOSI
- U1 pad 6: (no net) -> SCK
- U1 pad 7: (no net) -> HOLD
- U1 pad 8: (no net) -> 3V3
Routing:
- net (no net): track 1474.4 -> 1053.9 mm, vias 6 -> 0
- net GND: track 0.00 -> 107.1 mm, vias 0 -> 2
- net 3V3: track 0.00 -> 32.2 mm, vias 0 -> 1
- net MOSI: track 0.00 -> 21.2 mm, vias 0 -> 1
- net SCK: track 0.00 -> 18.8 mm, vias 0 -> 1
- net VBAT: track 0.00 -> 18.5 mm
- net WP: track 0.00 -> 17.0 mm
- net HOLD: track 0.00 -> 16.9 mm, vias 0 -> 1
- net 5V: track 0.00 -> 16.7 mm
- net MISO: track 0.00 -> 15.8 mm
- net CS: track 0.00 -> 15.3 mm
- net GENIO9: track 0.00 -> 9.78 mm
- net GENIO7: track 0.00 -> 9.78 mm
- net GENIO29: track 0.00 -> 9.78 mm
- net GENIO25: track 0.00 -> 9.78 mm
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Other:
- board text added: "HACKADAY SUPERCON 2019 BADGE CARTRIDGE (NO BLOWING INTO CONTACTS PLZKTHX)"
- board text added: "HDR1: 3V3 GND 3V3 GND 3V3 GND 3V3 GND IO1 IO2 IO3 IO4 IO5 IO6 .... IO29 IO30 5V VBAT"
- board text removed: "HACKADAY SUPERCON 2019 BADGE CARTRIDGE"
- board text removed: "HDR1: GND 3V3 NC NC NC NC NC NC IO2 IO1 IO4 IO3 IO5 IO4 .... IO30 IO29 5V VBAT"

Commit message: Add explanatory text for sidecart
Other:
- board text added: "Note: The main board is entirely hidden by (and has the same partial form factor as) the badge. The breakaway board on the side 'sticks out' on the right of the cart, and can be used to put user-interacting hardware on."
Changed lines of the file:
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@@
   (general
     (thickness 1.6)
-    (drawings 89)
+    (drawings 90)
     (tracks 275)
     (zones 0)
@@
     (47 F.CrtYd user hide)
     (48 B.Fab user)
-    (49 F.Fab user hide)
+    (49 F.Fab user)
   )
   (setup
@@
     )
   )
+  (gr_text "Note: The main board is entirely hidden by (and has \nthe same partial form factor as) the badge. The \nbreakaway board on the side 'sticks out' on the right of \nthe cart, and can be used to put user-interacting hardware \non." (at 148.2 92.8) (layer F.Fab)
+    (effects (font (size 1 1) (thickness 0.15)))
+  )
   (gr_line (start 110.67 66.37) (end 120.904 66.3575) (layer B.SilkS) (width 0.3))
